File: applications/TangNano6809MEM/rev1.0/TangNano6809MEM.kicad_pcb (KiCad board)
At the start: 2 copper layers, 73.7 x 73.7 mm, 22 parts, among them J1 TangNano20K5VInterface, J2 6809 TEST, J3 DBG, J4 HALT_n, J5 NMI_n, J6 IRQ_n, J7 FIRQ_n, J8 LED_RGB, U1 MC6809

Commit message: 6809MEM added
Parts:
- moved J4 7.62 mm to (5.08, 30.5)
- moved J7 7.62 mm to (5.08, 38.1)
- moved R4 7.62 mm to (20.3, 43.2)
- moved R6 7.62 mm to (20.3, 35.6)
- moved J5 2.54 mm to (5.08, 33.0)
- moved J6 2.54 mm to (5.08, 35.6)
- moved R2 2.54 mm to (20.3, 38.1)
- moved R3 2.54 mm to (20.3, 40.6)
Routing:
- net GND: track 131.1 -> 102.1 mm
- net PIN18: track 88.8 -> 71.4 mm, vias 1 -> 0
- net PIN19: track 82.6 -> 73.0 mm, vias 1 -> 0
- net FIRQ_n: track 35.3 -> 41.6 mm
- net PIN17: track 70.2 -> 76.4 mm, vias 1 -> 0
- net HALT_n: track 39.8 -> 34.0 mm
- net IRQ_n: track 31.3 -> 34.9 mm
- net PIN20: track 76.4 -> 74.5 mm, vias 1 -> 0
- net NMI_n: track 32.0 -> 30.2 mm
- net VCC: track 78.5 -> 79.5 mm
- net RW_n: track 85.6 -> 84.9 mm

Commit message: 6809MEM added
Parts:
- moved R1 9.16 mm to (7.62, 20.3), turned to 90 degrees
- moved R7 5.68 mm to (5.08, 20.3), turned to 90 degrees
- moved R5 2.54 mm to (2.54, 20.3), turned to 90 degrees
Routing:
- net GND: track 102.1 -> 150.8 mm
- net VCC: track 79.5 -> 71.9 mm, vias 1 -> 0
- net DMA_BREQ_n: track 30.1 -> 32.8 mm
- net MRDY: track 19.6 -> 22.3 mm
- net HALT_n: track 34.0 -> 32.1 mm
- net RESET_n: track 70.3 -> 72.1 mm
Other:
- board text added: "EXTAL (CLK)"
- board text added: "XTAL (GND)"
- board text removed: "CLK"
