File: applications/TangNano8008MEM/hardware/rev.1.0/TangNano8008MEM.kicad_sch (KiCad schematic)
At the start: 36 parts, among them J1 Barrel_Jack_Switch, J2 VCC_FPGA, J3 CPU Vcc, J4 TangNano20K5VInterface, J5 Conn_01x20, J6 Conn_01x20, J7 UART, SW1 SW_SPDT, U1 intel8008

Commit message: PCB for 8008 updated
Parts:
- removed C2: 0.1uF, 000_MyFootprint:C_Disc_D5.0mm_W2.5mm_P2.50mm, symbol 000_MyLibrary:C
- removed C3: 47uF, 000_MyFootprint:CP_Radial_D6.3mm_P2.50mm, symbol 000_MyLibrary:C_Polarized
- removed D1: LED, 000_MyFootprint:LED_D3.0mm, symbol 000_MyLibrary:LED
- removed J1: Barrel_Jack_Switch, 000_MyFootprint:BarrelJack_Horizontal, symbol 000_MyLibrary:Barrel_Jack_Switch
- removed J2: VCC_FPGA, 000_MyFootprint:PinHeader_1x02_P2.54mm_Vertical, symbol 000_MyLibrary:Conn_01x02_Male
- removed J3: CPU Vcc, 000_MyFootprint:PinHeader_1x03_P2.54mm_Vertical, symbol 000_MyLibrary:Conn_01x03_Male
- removed J5, J6: Conn_01x20, 000_MyFootprint:PinSocket_1x20_P2.54mm_Vertical, symbol 000_MyLibrary:Conn_01x20
- removed J7: UART, 000_MyFootprint:PinHeader_1x06_P2.54mm_Horizontal, symbol 000_MyLibrary:Conn_01x06_Pin
- removed R1: 100k, 000_MyFootprint:R_Axial_DIN0207_L6.3mm_D2.5mm_P7.62mm_Horizontal, symbol 000_MyLibrary:R
- removed R2, R3, R4: 1k, 000_MyFootprint:R_Axial_DIN0207_L6.3mm_D2.5mm_P7.62mm_Horizontal, symbol 000_MyLibrary:R
- removed SW1: SW_SPDT, 000_MyFootprint:SW_SPDT_Toggle_with_mount, symbol 000_MyLibrary:SW_SPDT
- added RN2: 1k, Resistor_THT:R_Array_SIP5, symbol 000_MyLibrary:R_Network04
- C1: renamed from C4; footprint 000_MyFootprint:CP_Radial_D6.3mm_P2.50mm -> 000_MyFootprint:CP_Radial_D5.0mm_P2.00mm
- C2: renamed from C1; footprint 000_MyFootprint:C_Disc_D5.0mm_W2.5mm_P2.50mm -> 000_MyFootprint:C_Disc_D4.7mm_W2.5mm_P5.00mm
- D1: renamed from D3; footprint (none) -> 000_MyFootprint:D_DO-35_SOD27_P2.54mm_Vertical_KathodeUp
- D2: renamed from D4; footprint (none) -> 000_MyFootprint:D_DO-35_SOD27_P2.54mm_Vertical_KathodeUp
- D3: renamed from D5; footprint (none) -> 000_MyFootprint:D_DO-35_SOD27_P2.54mm_Vertical_KathodeUp
- D4: renamed from D6; footprint (none) -> 000_MyFootprint:D_DO-35_SOD27_P2.54mm_Vertical_KathodeUp
- D5: renamed from D7; footprint (none) -> 000_MyFootprint:D_DO-35_SOD27_P2.54mm_Vertical_KathodeUp
- D6: renamed from D8; footprint (none) -> 000_MyFootprint:D_DO-35_SOD27_P2.54mm_Vertical_KathodeUp
- D7: renamed from D9; footprint (none) -> 000_MyFootprint:D_DO-35_SOD27_P2.54mm_Vertical_KathodeUp
- D8: renamed from D10; footprint (none) -> 000_MyFootprint:D_DO-35_SOD27_P2.54mm_Vertical_KathodeUp
- U1: footprint (none) -> 000_MyFootprint:DIP_Socket-18_W4.3_W5.08_W7.62_W10.16_W10.9_3M_218-3341-00-0602J
- renumbered D2 to D9, J4 to J1, R7 to R1, R8 to R2, R9 to R3, R10 to R4, RN2 to RN3
Connections:
- net VCC_FPGA is gone; now on net +5V: J1.40 (Pin_40)
- net +5V: now also RN2.1 (common); no longer R5.2
- net -9V: now also R5.2
- net CLK1: now also RN2.4 (R3)
- net CLK2: now also RN2.5 (R4); no longer R5.1
- net D0: now also D8.1 (K), RN1.9 (R8); no longer D1.1 (K), RN1.2 (R1)
- net D1: now also D7.1 (K), RN1.8 (R7); no longer D2.1 (K), RN1.3 (R2)
- net D2: now also D6.1 (K), RN1.7 (R6); no longer D3.1 (K), RN1.4 (R3)
- net D3: now also D5.1 (K), RN1.6 (R5); no longer D4.1 (K), RN1.5 (R4)
- net D4: now also D4.1 (K), RN1.5 (R4); no longer D5.1 (K), RN1.6 (R5)
- net D5: now also D3.1 (K), RN1.4 (R3); no longer D6.1 (K), RN1.7 (R6)
- net D6: now also D2.1 (K), RN1.3 (R2); no longer D7.1 (K), RN1.8 (R7)
- net D7: now also D1.1 (K), RN1.2 (R1); no longer D8.1 (K), RN1.9 (R8)
- net GND: now also R5.1
- net INTERRUPT: now also RN2.2 (R1)
- net READY: now also RN2.3 (R2)
- no-connect marks 5 -> 8
Other:
- note removed: "DC Jack"
- note removed: "RX<-TX"
- note removed: "Select CPU's Vcc source connect 1-2: DC Jack connect 2-3: USB (FPGA's Vcc)"
- note removed: "Select FPGA's Vcc source open: USB connect 1-2: DC Jack"
- note removed: "TX->RX"
- note removed: "USB"
- moved on the sheet: C1, C2, D9, J1, PS1, R6
